Commit message: oprava

File: description/ros2_control_sim.xacro (robot description, xacro)
@@ -18,5 +18,5 @@
     <state_interface name="acceleration"/>
   </joint>
-  <joint name="front_reight_wheel_joint">
+  <joint name="front_right_wheel_joint">
     <command_interface name="velocity"/>
     <command_interface name="acceleration"/>
@@ -37,5 +37,5 @@
     <state_interface name="acceleration"/>
   </joint>
-  <joint name="rear_reight_wheel_joint">
+  <joint name="rear_right_wheel_joint">
     <command_interface name="velocity"/>
     <command_interface name="acceleration"/>

Commit message: joint

File: description/ros2_control_sim.xacro (robot description, xacro)
@@ -9,5 +9,5 @@
     <param name="position_state_following_offset">0.0</param>
   </hardware>
-  <joint name="front_left_wheel_joint">
+  <joint name="joint1">
     <command_interface name="position"/>
     <command_interface name="velocity"/>
@@ -18,5 +18,5 @@
     <state_interface name="acceleration"/>
   </joint>
-  <joint name="front_right_wheel_joint">
+  <joint name="joint2">
     <command_interface name="velocity"/>
     <command_interface name="acceleration"/>
@@ -28,5 +28,5 @@
     <state_interface name="acceleration"/>
   </joint>
-  <joint name="rear_left_wheel_joint">
+  <joint name="joint3">
     <command_interface name="position"/>
     <command_interface name="velocity"/>
@@ -37,5 +37,5 @@
     <state_interface name="acceleration"/>
   </joint>
-  <joint name="rear_right_wheel_joint">
+  <joint name="joint4">
     <command_interface name="velocity"/>
     <command_interface name="acceleration"/>
