Commit message: real robot

File: description/robot.urdf.xacro (robot description, xacro)
@@ -4,4 +4,4 @@
     <xacro:include filename="lidar.xacro" />
     <xacro:arg name="use_ros2_control" default="true"/>
-    <xacro:include filename="ros2_control_sim.xacro" />
+    <xacro:include filename="ros2_control.xacro" />
 </robot>

File: description/ros2_control_sim.xacro (robot description, xacro)
@@ -9,5 +9,5 @@
     <param name="position_state_following_offset">0.0</param>
   </hardware>
-  <joint name="joint1">
+  <joint name="front_left_wheel_joint">
     <command_interface name="position"/>
     <command_interface name="velocity"/>
@@ -18,5 +18,5 @@
     <state_interface name="acceleration"/>
   </joint>
-  <joint name="joint2">
+  <joint name="front_right_wheel_joint">
     <command_interface name="velocity"/>
     <command_interface name="acceleration"/>
@@ -28,5 +28,5 @@
     <state_interface name="acceleration"/>
   </joint>
-  <joint name="joint3">
+  <joint name="rear_left_wheel_joint">
     <command_interface name="position"/>
     <command_interface name="velocity"/>
@@ -37,5 +37,5 @@
     <state_interface name="acceleration"/>
   </joint>
-  <joint name="joint4">
+  <joint name="rear_right_wheel_joint">
     <command_interface name="velocity"/>
     <command_interface name="acceleration"/>
