Commit message: odebrani xacro:inertial_cylinder

File: description/lidar.xacro (robot description, xacro)
@@ -25,7 +25,4 @@
             </geometry>
         </collision>
-        <xacro:inertial_cylinder mass="0.1" length="0.04" radius="0.05">
-            <origin xyz="0 0 0" rpy="0 0 0"/>
-        </xacro:inertial_cylinder>
     </link>
 </robot>

Commit message: laser_frame fix

File: description/lidar.xacro (robot description, xacro)
@@ -4,5 +4,5 @@
         <parent link="chassis"/>
         <child link="laser_frame"/>
-        <origin xyz="0.122 0 0.212" rpy="0 0 0"/>
+        <origin xyz="0 0 0" rpy="0 0 0"/>
     </joint>
     <link name="laser_frame">

Commit message: změny urdf

File: description/lidar.xacro (robot description, xacro)
@@ -1,5 +1,5 @@
 <?xml version="1.0"?>
 <robot xmlns:xacro="http://www.ros.org/wiki/xacro" >
-    <joint name="laser_joint" type="fixed">
+    <!-- <joint name="laser_joint" type="fixed">
         <parent link="chassis"/>
         <child link="laser_frame"/>
@@ -25,4 +25,49 @@
             </geometry>
         </collision>
+    </link> -->
+    <!-- ===== LiDAR 1 ===== -->
+    <link name="laser_frame1">
+        <visual>
+            <geometry>
+                <cylinder radius="0.055" length="0.04"/>
+            </geometry>
+            <material name="black"/>
+        </visual>
+        <visual>
+            <origin xyz="0 0 -0.05"/>
+            <geometry>
+                <cylinder radius="0.01" length="0.1"/>
+            </geometry>
+            <material name="black"/>
+        </visual>
     </link>
+  <joint name="base_to_lidar1" type="fixed">
+    <parent link="base_link"/>
+    <child link="laser_frame1"/>
+    <!-- TODO: doplň reálné hodnoty v metrech a radiánech -->
+    <!-- xyz: dopředu +x, doleva +y, nahoru +z (REP-103) -->
+    <origin xyz="0.2705 0.332 0.45" rpy="0 0 3.14159265359"/>
+  </joint>
+  <!-- ===== LiDAR 2 ===== -->
+    <link name="laser_frame2">
+        <visual>
+            <geometry>
+                <cylinder radius="0.055" length="0.04"/>
+            </geometry>
+            <material name="black"/>
+            </visual>
+            <visual>
+                <origin xyz="0 0 -0.05"/>
+                <geometry>
+                    <cylinder radius="0.01" length="0.1"/>
+                </geometry>
+                <material name="black"/>
+            </visual>
+        </link>
+  <joint name="base_to_lidar2" type="fixed">
+    <parent link="base_link"/>
+    <child link="laser_frame2"/>
+    <!-- TODO: doplň reálné hodnoty -->
+    <origin xyz="-0.2705 -0.332 0.45" rpy="0 0 0"/>
+  </joint>
 </robot>

File: description/robot_core.xacro (robot description, xacro)
@@ -2,6 +2,6 @@
 <robot xmlns:xacro="http://www.ros.org/wiki/xacro" >
     <xacro:include filename="inertial_macros.xacro"/>
-    <xacro:property name="chassis_length" value="0.63"/>
-    <xacro:property name="chassis_width" value="0.72"/>
+    <xacro:property name="chassis_length" value="0.560"/>
+    <xacro:property name="chassis_width" value="0.560"/>
     <xacro:property name="chassis_height" value="0.5"/>
     <xacro:property name="chassis_mass" value="1.0"/>
@@ -9,7 +9,7 @@
     <xacro:property name="wheel_thickness" value="0.034"/>
     <xacro:property name="wheel_mass" value="0.05"/>
-    <xacro:property name="wheel_offset_x" value="0.192"/>
-    <xacro:property name="wheel_offset_y" value="0.262"/>
-    <xacro:property name="wheel_offset_z" value="0.026"/>
+    <xacro:property name="wheel_offset_x" value="0.2035"/>
+    <xacro:property name="wheel_offset_y" value="0.253"/>
+    <xacro:property name="wheel_offset_z" value="0.052"/>
     <xacro:property name="caster_wheel_radius" value="0.01"/>
     <xacro:property name="caster_wheel_mass" value="0.01"/>

Commit message: oprava

File: description/lidar.xacro (robot description, xacro)
@@ -27,4 +27,11 @@
     </link> -->
     <!-- ===== LiDAR 1 ===== -->
+    <joint name="base_to_lidar1" type="fixed">
+    <parent link="chassis"/>
+    <child link="laser_frame1"/>
+    <!-- TODO: doplň reálné hodnoty v metrech a radiánech -->
+    <!-- xyz: dopředu +x, doleva +y, nahoru +z (REP-103) -->
+    <origin xyz="0.2705 0.332 0.45" rpy="0 0 3.14159265359"/>
+  </joint>
     <link name="laser_frame1">
         <visual>
@@ -37,17 +44,16 @@
             <origin xyz="0 0 -0.05"/>
             <geometry>
-                <cylinder radius="0.01" length="0.1"/>
+                <cylinder radius="0.055" length="0.04"/>
             </geometry>
             <material name="black"/>
         </visual>
     </link>
-  <joint name="base_to_lidar1" type="fixed">
-    <parent link="base_link"/>
-    <child link="laser_frame1"/>
-    <!-- TODO: doplň reálné hodnoty v metrech a radiánech -->
-    <!-- xyz: dopředu +x, doleva +y, nahoru +z (REP-103) -->
-    <origin xyz="0.2705 0.332 0.45" rpy="0 0 3.14159265359"/>
+  <!-- ===== LiDAR 2 ===== -->
+  <joint name="base_to_lidar2" type="fixed">
+    <parent link="chassis"/>
+    <child link="laser_frame2"/>
+    <!-- TODO: doplň reálné hodnoty -->
+    <origin xyz="-0.2705 -0.332 0.45" rpy="0 0 0"/>
   </joint>
-  <!-- ===== LiDAR 2 ===== -->
     <link name="laser_frame2">
         <visual>
@@ -60,14 +66,8 @@
                 <origin xyz="0 0 -0.05"/>
                 <geometry>
-                    <cylinder radius="0.01" length="0.1"/>
+                    <cylinder radius="0.055" length="0.04"/>
                 </geometry>
                 <material name="black"/>
             </visual>
         </link>
-  <joint name="base_to_lidar2" type="fixed">
-    <parent link="base_link"/>
-    <child link="laser_frame2"/>
-    <!-- TODO: doplň reálné hodnoty -->
-    <origin xyz="-0.2705 -0.332 0.45" rpy="0 0 0"/>
-  </joint>
 </robot>

Commit message: pokus

File: description/lidar.xacro (robot description, xacro)
@@ -1,5 +1,5 @@
 <?xml version="1.0"?>
 <robot xmlns:xacro="http://www.ros.org/wiki/xacro" >
-    <!-- <joint name="laser_joint" type="fixed">
+    <joint name="laser_joint" type="fixed">
         <parent link="chassis"/>
         <child link="laser_frame"/>
@@ -25,13 +25,11 @@
             </geometry>
         </collision>
-    </link> -->
-    <!-- ===== LiDAR 1 ===== -->
+    </link>
+    <!--
     <joint name="base_to_lidar1" type="fixed">
-    <parent link="chassis"/>
+    <parent link="base_link"/>
     <child link="laser_frame1"/>
-    <!-- TODO: doplň reálné hodnoty v metrech a radiánech -->
-    <!-- xyz: dopředu +x, doleva +y, nahoru +z (REP-103) -->
     <origin xyz="0.2705 0.332 0.45" rpy="0 0 3.14159265359"/>
-  </joint>
+    </joint>
     <link name="laser_frame1">
         <visual>
@@ -49,11 +47,9 @@
         </visual>
     </link>
-  <!-- ===== LiDAR 2 ===== -->
-  <joint name="base_to_lidar2" type="fixed">
-    <parent link="chassis"/>
+    <joint name="base_to_lidar2" type="fixed">
+    <parent link="base_link"/>
     <child link="laser_frame2"/>
-    <!-- TODO: doplň reálné hodnoty -->
     <origin xyz="-0.2705 -0.332 0.45" rpy="0 0 0"/>
-  </joint>
+    </joint>
     <link name="laser_frame2">
         <visual>
@@ -71,3 +67,4 @@
             </visual>
         </link>
+-->
 </robot>

Commit message: oprava

File: description/lidar.xacro (robot description, xacro)
@@ -1,4 +1,5 @@
 <?xml version="1.0"?>
 <robot xmlns:xacro="http://www.ros.org/wiki/xacro" >
+<!--
     <joint name="laser_joint" type="fixed">
         <parent link="chassis"/>
@@ -7,4 +8,55 @@
     </joint>
     <link name="laser_frame">
+        <visual>
+            <geometry>
+                <cylinder radius="0.05" length="0.04"/>
+            </geometry>
+            <material name="black"/>
+        </visual>
+        <visual>
+            <origin xyz="0 0 -0.05"/>
+            <geometry>
+                <cylinder radius="0.01" length="0.1"/>
+            </geometry>
+            <material name="black"/>
+        </visual>
+        <collision>
+            <geometry>
+                <cylinder radius="0.05" length="0.04"/>
+            </geometry>
+        </collision>
+    </link>
+-->
+    <joint name="laser_joint" type="fixed">
+        <parent link="chassis"/>
+        <child link="laser_frame"/>
+        <origin xyz="0.2705 0.332 0.45" rpy="0 0 3.1415"/>
+    </joint>
+    <link name="laser_frame">
+        <visual>
+            <geometry>
+                <cylinder radius="0.05" length="0.04"/>
+            </geometry>
+            <material name="black"/>
+        </visual>
+        <visual>
+            <origin xyz="0 0 -0.05"/>
+            <geometry>
+                <cylinder radius="0.01" length="0.1"/>
+            </geometry>
+            <material name="black"/>
+        </visual>
+        <collision>
+            <geometry>
+                <cylinder radius="0.05" length="0.04"/>
+            </geometry>
+        </collision>
+    </link>
+    <joint name="laser_joint2" type="fixed">
+        <parent link="chassis"/>
+        <child link="laser_frame2"/>
+        <origin xyz="-0.2705 -0.332 0.45" rpy="0 0 0"/>
+    </joint>
+    <link name="laser_frame2">
         <visual>
             <geometry>

Commit message: obrácení lidaru

File: description/lidar.xacro (robot description, xacro)
@@ -31,5 +31,5 @@
         <parent link="chassis"/>
         <child link="laser_frame"/>
-        <origin xyz="0.2705 0.332 0.45" rpy="0 0 3.1415"/>
+        <origin xyz="0.2705 0.332 0.45" rpy="0 0 0"/>
     </joint>
     <link name="laser_frame">

Commit message: lidar

File: description/lidar.xacro (robot description, xacro)
@@ -31,5 +31,5 @@
         <parent link="chassis"/>
         <child link="laser_frame"/>
-        <origin xyz="0.2705 0.332 0.45" rpy="0 0 0"/>
+        <origin xyz="0.2705 0.332 0.45" rpy="0 0 3.1415"/>
     </joint>
     <link name="laser_frame">

Commit message: otočení lidaru zpátky

File: description/lidar.xacro (robot description, xacro)
@@ -31,5 +31,5 @@
         <parent link="chassis"/>
         <child link="laser_frame"/>
-        <origin xyz="0.2705 0.332 0.45" rpy="0 0 0"/>
+        <origin xyz="0.2705 0.332 0.45" rpy="0 0 3.141592"/>
     </joint>
     <link name="laser_frame">
