Commit message: pokus axis

File: description/robot_core.xacro (robot description, xacro)
@@ -70,5 +70,5 @@
         <child link="front_left_wheel"/>
         <origin xyz="${wheel_offset_x} ${wheel_offset_y} 0" rpy="-${pi/2} 0 0" />
-        <axis xyz="0 0 1"/>
+        <axis xyz="0 0 -1"/>
     </joint>
     <link name="front_left_wheel">
@@ -93,5 +93,5 @@
         <child link="front_right_wheel"/>
         <origin xyz="${wheel_offset_x} ${-wheel_offset_y} 0" rpy="${pi/2} 0 0" />
-        <axis xyz="0 0 -1"/>
+        <axis xyz="0 0 1"/>
     </joint>
     <link name="front_right_wheel">
@@ -116,5 +116,5 @@
         <child link="rear_left_wheel"/>
         <origin xyz="${-wheel_offset_x} ${wheel_offset_y} 0" rpy="-${pi/2} 0 0" />
-        <axis xyz="0 0 1"/>
+        <axis xyz="0 0 -1"/>
     </joint>
     <link name="rear_left_wheel">
@@ -139,5 +139,5 @@
         <child link="rear_right_wheel"/>
         <origin xyz="${-wheel_offset_x} ${-wheel_offset_y} 0" rpy="${pi/2} 0 0" />
-        <axis xyz="0 0 -1"/>
+        <axis xyz="0 0 1"/>
     </joint>
     <link name="rear_right_wheel">

Commit message: obrácení hodnot

File: description/robot_core.xacro (robot description, xacro)
@@ -70,5 +70,5 @@
         <child link="front_left_wheel"/>
         <origin xyz="${wheel_offset_x} ${wheel_offset_y} 0" rpy="-${pi/2} 0 0" />
-        <axis xyz="0 0 -1"/>
+        <axis xyz="0 0 1"/>
     </joint>
     <link name="front_left_wheel">
@@ -93,5 +93,5 @@
         <child link="front_right_wheel"/>
         <origin xyz="${wheel_offset_x} ${-wheel_offset_y} 0" rpy="${pi/2} 0 0" />
-        <axis xyz="0 0 1"/>
+        <axis xyz="0 0 -1"/>
     </joint>
     <link name="front_right_wheel">
@@ -116,5 +116,5 @@
         <child link="rear_left_wheel"/>
         <origin xyz="${-wheel_offset_x} ${wheel_offset_y} 0" rpy="-${pi/2} 0 0" />
-        <axis xyz="0 0 -1"/>
+        <axis xyz="0 0 1"/>
     </joint>
     <link name="rear_left_wheel">
@@ -139,5 +139,5 @@
         <child link="rear_right_wheel"/>
         <origin xyz="${-wheel_offset_x} ${-wheel_offset_y} 0" rpy="${pi/2} 0 0" />
-        <axis xyz="0 0 1"/>
+        <axis xyz="0 0 -1"/>
     </joint>
     <link name="rear_right_wheel">

Commit message: test

File: description/robot_core.xacro (robot description, xacro)
@@ -9,6 +9,6 @@
     <xacro:property name="wheel_thickness" value="0.026"/>
     <xacro:property name="wheel_mass" value="0.05"/>
-    <xacro:property name="wheel_offset_x" value="0.265"/>
-    <xacro:property name="wheel_offset_y" value="0.315"/>
+    <xacro:property name="wheel_offset_x" value="0.192"/>
+    <xacro:property name="wheel_offset_y" value="0.287"/>
     <xacro:property name="wheel_offset_z" value="0.01"/>
     <xacro:property name="caster_wheel_radius" value="0.01"/>

Commit message: zmena velikosti kola

File: description/robot_core.xacro (robot description, xacro)
@@ -2,10 +2,10 @@
 <robot xmlns:xacro="http://www.ros.org/wiki/xacro" >
     <xacro:include filename="inertial_macros.xacro"/>
-    <xacro:property name="chassis_length" value="0.53"/>
-    <xacro:property name="chassis_width" value="0.55"/>
-    <xacro:property name="chassis_height" value="1.0"/>
+    <xacro:property name="chassis_length" value="0.4"/>
+    <xacro:property name="chassis_width" value="0.4"/>
+    <xacro:property name="chassis_height" value="0.5"/>
     <xacro:property name="chassis_mass" value="1.0"/>
-    <xacro:property name="wheel_radius" value="0.055"/>
-    <xacro:property name="wheel_thickness" value="0.026"/>
+    <xacro:property name="wheel_radius" value="0.052"/>
+    <xacro:property name="wheel_thickness" value="0.034"/>
     <xacro:property name="wheel_mass" value="0.05"/>
     <xacro:property name="wheel_offset_x" value="0.192"/>

Commit message: ZMENA MODELU

File: description/robot_core.xacro (robot description, xacro)
@@ -10,6 +10,6 @@
     <xacro:property name="wheel_mass" value="0.05"/>
     <xacro:property name="wheel_offset_x" value="0.192"/>
-    <xacro:property name="wheel_offset_y" value="0.287"/>
-    <xacro:property name="wheel_offset_z" value="0.01"/>
+    <xacro:property name="wheel_offset_y" value="0.262"/>
+    <xacro:property name="wheel_offset_z" value="0.026"/>
     <xacro:property name="caster_wheel_radius" value="0.01"/>
     <xacro:property name="caster_wheel_mass" value="0.01"/>

Commit message: uprava tf

File: description/robot_core.xacro (robot description, xacro)
@@ -2,6 +2,6 @@
 <robot xmlns:xacro="http://www.ros.org/wiki/xacro" >
     <xacro:include filename="inertial_macros.xacro"/>
-    <xacro:property name="chassis_length" value="0.4"/>
-    <xacro:property name="chassis_width" value="0.4"/>
+    <xacro:property name="chassis_length" value="0.63"/>
+    <xacro:property name="chassis_width" value="0.72"/>
     <xacro:property name="chassis_height" value="0.5"/>
     <xacro:property name="chassis_mass" value="1.0"/>
@@ -69,5 +69,5 @@
         <parent link="base_link"/>
         <child link="front_left_wheel"/>
-        <origin xyz="${wheel_offset_x} ${wheel_offset_y} 0" rpy="-${pi/2} 0 0" />
+        <origin xyz="${wheel_offset_x} ${wheel_offset_y} ${wheel_offset_z}" rpy="-${pi/2} 0 0" />
         <axis xyz="0 0 1"/>
     </joint>
@@ -92,5 +92,5 @@
         <parent link="base_link"/>
         <child link="front_right_wheel"/>
-        <origin xyz="${wheel_offset_x} ${-wheel_offset_y} 0" rpy="${pi/2} 0 0" />
+        <origin xyz="${wheel_offset_x} ${-wheel_offset_y} ${wheel_offset_z}" rpy="${pi/2} 0 0" />
         <axis xyz="0 0 -1"/>
     </joint>
@@ -115,5 +115,5 @@
         <parent link="base_link"/>
         <child link="rear_left_wheel"/>
-        <origin xyz="${-wheel_offset_x} ${wheel_offset_y} 0" rpy="-${pi/2} 0 0" />
+        <origin xyz="${-wheel_offset_x} ${wheel_offset_y} ${wheel_offset_z}" rpy="-${pi/2} 0 0" />
         <axis xyz="0 0 1"/>
     </joint>
@@ -138,5 +138,5 @@
         <parent link="base_link"/>
         <child link="rear_right_wheel"/>
-        <origin xyz="${-wheel_offset_x} ${-wheel_offset_y} 0" rpy="${pi/2} 0 0" />
+        <origin xyz="${-wheel_offset_x} ${-wheel_offset_y} ${wheel_offset_z}" rpy="${pi/2} 0 0" />
         <axis xyz="0 0 -1"/>
     </joint>

Commit message: přidání imu

File: description/robot_core.xacro (robot description, xacro)
@@ -33,4 +33,20 @@
     <link name="base_link">
     </link>
+    <!-- IMU frame -->
+    <link name="imu_link">
+    <!-- vizuál/kolize jsou volitelné; pro TF stačí samotný link -->
+    <inertial>
+        <origin xyz="0 0 0" rpy="0 0 0"/>
+        <mass value="0.01"/>
+        <inertia ixx="1e-6" ixy="0" ixz="0" iyy="1e-6" iyz="0" izz="1e-6"/>
+    </inertial>
+    </link>
+    <!-- Fixed transform base_link -> imu_link -->
+    <joint name="base_to_imu" type="fixed">
+    <parent link="base_link"/>
+    <child link="imu_link"/>
+    <!-- Umístění IMU vůči base_link (v metrech) -->
+    <origin xyz="0.055 -0.033 0.21" rpy="0 0 0"/>
+    </joint>
      <!-- BASE_FOOTPRINT LINK -->
     <joint name="base_footprint_joint" type="fixed">

Commit message: oprava

File: description/robot_core.xacro (robot description, xacro)
@@ -47,5 +47,5 @@
     <child link="imu_link"/>
     <!-- Umístění IMU vůči base_link (v metrech) -->
-    <origin xyz="0.055 -0.033 0.21" rpy="0 0 0"/>
+    <origin xyz="0.055 -0.33 0.21" rpy="0 0 0"/>
     </joint>
      <!-- BASE_FOOTPRINT LINK -->

Commit message: uprava pro lineární posun

File: description/robot_core.xacro (robot description, xacro)
@@ -173,3 +173,21 @@
         </xacro:inertial_cylinder>
     </link>
+    <!-- Lineární vozík / posuvný díl -->
+    <link name="linear_carriage_link">
+    <inertial>
+        <mass value="0.5"/>
+        <origin xyz="0 0 0" rpy="0 0 0"/>
+        <inertia ixx="0.001" ixy="0" ixz="0" iyy="0.001" iyz="0" izz="0.001"/>
+    </inertial>
+    </link>
+    <!-- Prismatic joint pro lineární posun -->
+    <joint name="linear_axis_joint" type="prismatic">
+    <parent link="base_link"/>
+    <child link="linear_carriage_link"/>
+    <!-- osa posuvu (uprav podle reality) -->
+    <axis xyz="1 0 0"/>
+    <!-- limity v metrech + max rychlost (m/s) -->
+    <limit lower="0.0" upper="0.20" effort="50" velocity="0.05"/>
+    <origin xyz="0 0 0" rpy="0 0 0"/>
+    </joint>
 </robot>

File: description/ros2_control.xacro (robot description, xacro)
@@ -13,4 +13,8 @@
             <param name="timeout_ms">1000</param>
             <param name="enc_counts_per_rev">1350</param>
+            <param name="enable_linear_axis">true</param>
+            <param name="linear_axis_name">linear_axis_joint</param>
+            <!-- pokud děláš prismatic joint v metrech: m / encoder_count -->
+            <param name="linear_axis_units_per_count">0.0000125</param>
         </hardware>
         <joint name="front_left_wheel_joint">
@@ -46,4 +50,9 @@
             <state_interface name="velocity"/>
         </joint>
+        <joint name="linear_axis_joint">
+            <command_interface name="velocity"/>
+            <state_interface name="position"/>
+            <state_interface name="velocity"/>
+        </joint>
     </ros2_control>
 </robot>
